File: eagle/badge2016.sch (EAGLE design)
At the start: 82 parts, among them IC1 FT230XS, IC3 24AA01SN, J1 USB-MICRO, Q2 BC857ALT1SMD, X1 PASSER-07, X2 PASSER-07, X3 PASSER-07

Commit message: Update badge2016.sch
Review and changes LTC3554:
* Missing connecting Pin 9 (PWR_ON1) via R11 to Pin 18 (V_OUT) to activate SW1
* Change R2 from 1.87k to 750 (for max. load of 1A)
* PIN 15 (NTC) to GND, because NTC is not in use
Parts:
- R2: value 1.87k -> 750
Connections:
- removed net N$24: R11.1
- net GND: now also U$11.NTC
- net V_USB: now also R11.1
Changed lines of the file:
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@@
 <part name="GND21" library="supply1" deviceset="GND" device=""/>
 <part name="U$11" library="ERNW_parts" deviceset="LTC3554" device=""/>
-<part name="R2" library="rcl" deviceset="R-EU_" device="R0402" value="1.87k"/>
+<part name="R2" library="rcl" deviceset="R-EU_" device="R0402" value="750"/>
 <part name="GND22" library="supply1" deviceset="GND" device=""/>
 <part name="C23" library="rcl" deviceset="C-EU" device="C0805" value="10µF"/>
@@
 <part name="JP4" library="pinhead" deviceset="PINHD-2X8" device=""/>
 <part name="GND51" library="supply1" deviceset="GND" device=""/>
+<part name="GND44" library="supply1" deviceset="GND" device=""/>
 </parts>
 <sheets>
@@
 <instance part="JP4" gate="A" x="-63.5" y="266.7"/>
 <instance part="GND51" gate="1" x="-93.98" y="266.7" rot="R270"/>
+<instance part="GND44" gate="1" x="50.8" y="-325.12" rot="R90"/>
 </instances>
 <busses>
@@
 <wire x1="-185.42" y1="27.94" x2="-185.42" y2="20.32" width="0.1524" layer="91"/>
 <junction x="-185.42" y="27.94"/>
-</segment>
-<segment>
-<pinref part="R2" gate="G$1" pin="2"/>
-<pinref part="GND22" gate="1" pin="GND"/>
-<wire x1="27.94" y1="-287.02" x2="27.94" y2="-281.94" width="0.1524" layer="91"/>
 </segment>
 <segment>
@@
 <wire x1="-91.44" y1="266.7" x2="-78.74" y2="266.7" width="0.1524" layer="91"/>
 </segment>
+<segment>
+<pinref part="GND44" gate="1" pin="GND"/>
+<pinref part="U$11" gate="G$1" pin="NTC"/>
+<wire x1="48.26" y1="-325.12" x2="45.72" y2="-325.12" width="0.1524" layer="91"/>
+</segment>
+<segment>
+<pinref part="GND22" gate="1" pin="GND"/>
+<pinref part="R2" gate="G$1" pin="2"/>
+<wire x1="27.94" y1="-281.94" x2="27.94" y2="-287.02" width="0.1524" layer="91"/>
+</segment>
 </net>
 <net name="3V3" class="0">
@@
 <pinref part="L2" gate="G$1" pin="1"/>
 <wire x1="60.96" y1="-327.66" x2="63.5" y2="-327.66" width="0.1524" layer="91"/>
-</segment>
-</net>
-<net name="N$24" class="0">
-<segment>
-<pinref part="R11" gate="G$1" pin="1"/>
-<wire x1="25.4" y1="-378.46" x2="25.4" y2="-388.62" width="0.1524" layer="91"/>
-<label x="25.4" y="-388.62" size="1.778" layer="95" rot="R90"/>
 </segment>
 </net>
@@
 <junction x="55.88" y="-271.78"/>
 <label x="38.1" y="-271.78" size="1.778" layer="95"/>
-</segment>
-<segment>
+<pinref part="R11" gate="G$1" pin="1"/>
+<wire x1="25.4" y1="-378.46" x2="25.4" y2="-381" width="0.1524" layer="91"/>
+<wire x1="25.4" y1="-381" x2="58.42" y2="-381" width="0.1524" layer="91"/>
+<wire x1="58.42" y1="-381" x2="58.42" y2="-332.74" width="0.1524" layer="91"/>
+</segment>
+<segment>

Commit message: New Display New USB <-> Serial + Connection to Power Supply Chip Moved Power Supply Chip, UART und JTAG Headers Changed Expansion Header
Parts:
- removed BAT: (no value), pinhead:PINHD-1X2
- removed IC1: FT230XS, ftdichip:FT230XS
- removed R15, R18: 100k, rcl:R-EU_R0402
- added C35: 100nF, rcl:C-EUC0402
- added C36: 4.7µF, rcl:C-EUC0402
- added R19: 4k32, rcl:R-EU_R0402
- added R20: 1k5, rcl:R-EU_R0402
- added SD1: SD-CARD-MSD50, we-con:SD-CARD-MSD50
- added U$14: MI0283QT, ERNW_parts:MI0283QT
- added U$15: JST-2, ERNW_parts:JST-2
- C31: value 100nF -> 4.7µF
- C32: value 4.7µF -> 100nF
- R2: value 750 -> 16k5
- U$12: value SAINSMART_2.4_TFT -> FT231X; device ERNW_parts:SAINSMART_2.4_TFT -> ERNW_parts:FT231X
Connections:
- removed net CS: U$1.DIO_11, U$12.CS
- removed net DB10: U$1.DIO_5, U$12.DB10
- removed net DB11: U$1.DIO_6, U$12.DB11
- removed net DB12: U$1.DIO_7, U$12.DB12
- removed net DB13: U$1.DIO_8, U$12.DB13
- removed net DB14: U$1.DIO_9, U$12.DB14
- removed net DB15: U$1.DIO_10, U$12.DB15
- removed net DB8: U$1.DIO_3, U$12.DB8
- removed net DB9: U$1.DIO_4, U$12.DB9
- removed net N$16: R2.1, U$11.PROG
- removed net N$19: C30.2, IC1.!RESET, IC1.3V3OUT, IC1.VCCIO
- removed net N$21: R18.2, U$1.DIO_22
- removed net N$31: R15.1, U$1.DIO_24
- removed net REST: U$1.DIO_12, U$12.REST
- removed net RS: U$1.DIO_1, U$12.RS
- removed net SD_CS: U$1.DIO_21, U$12.SD_CS
- removed net T_CS: U$1.DIO_13, U$12.T_CS
- removed net T_IRQ: U$1.DIO_14, U$12.T_IRQ
- removed net WR: U$1.DIO_2, U$12.WR
- new net !BCD: R20.2, U$12.CBUS0
- new net !PWREN: R19.1, U$12.CBUS1
- new net !SLEEP: U$11.SUSP, U$12.CBUS2
- new net D_!CS: U$1.DIO_13, U$14.!CS
- new net D_!RST: U$1.DIO_14, U$14.!RST
- new net D_ADS_!CS: U$1.DIO_12, U$14.!ADS-CS
- new net D_AUX: U$14.AUX
- new net D_BUSY: U$1.DIO_10, U$14.BUSY
- new net D_IRQ: U$1.DIO_11, U$14.IRQ
- new net IO3: JP4.6, U$1.DIO_26
- new net IO4: JP4.8, U$1.DIO_27
- new net IO5: JP4.10, U$1.DIO_28
- new net N$24: U$14.VREF
- new net N$26: U$14.VBAT
- new net N$34: U$1.DIO_8
- new net N$35: U$1.DIO_9
- new net N$37: C32.2, U$12.!RESET, U$12.3V3OUT, U$12.VCCIO
- new net N$46: SD1.DAT1
- new net N$47: SD1.DAT2
- new net PROG: R19.2, R2.1, R20.1, U$11.PROG
- new net SD_!CS: SD1.!CS
- new net SD_SWITCH: SD1.SW2
- net 3V3: now also C35.2, C36.2, SD1.3V3
- net DM: now also U$12.USBDM; no longer IC1.USBDM
- net DP: now also U$12.USBDP; no longer IC1.USBDP
- net GND: now also C30.2, C32.1, C35.1, C36.1, SD1.GND, SD1.SW1, U$12.GND0, U$12.GND1, U$12.GND2, U$14.GND0, U$14.GND1, U$15.P$1; no longer BAT.1, C30.1, C32.2, IC1.GND, IC1.GND@1, U$12.DB0, U$12.DB1, U$12.DB2, U$12.DB3, U$12.DB4, U$12.DB5, U$12.DB6, U$12.DB7, U$12.GND
- net I2C_SCL: now also JP4.14, U$1.DIO_20; no longer JP4.16, U$1.DIO_27
- net I2C_SDA: now also JP4.16, U$1.DIO_21; no longer JP4.14, U$1.DIO_28
- net IO1: now also JP4.2, U$1.DIO_24; no longer JP4.8, U$1.DIO_25
- net IO2: now also JP4.4, U$1.DIO_25; no longer JP4.10, U$1.DIO_26
- net LED_A: now also U$14.LED; no longer U$12.LED_A
- net N$20: now also U$15.P$2; no longer BAT.2
- net RXD: now also U$1.DIO_19, U$12.RXD; no longer IC1.RXD, U$1.DIO_29
- net SPI_CLK: now also SD1.SCK, U$1.DIO_6, U$14.SCK; no longer JP4.6, U$1.DIO_18, U$12.SD_CLK, U$12.T_CLK
- net SPI_MISO: now also SD1.MISO, U$1.DIO_5, U$14.MISO; no longer JP4.2, U$1.DIO_20, U$12.SD_DO, U$12.T_DO
- net SPI_MOSI: now also SD1.MOSI, U$1.DIO_7, U$14.MOSI; no longer JP4.4, U$1.DIO_19, U$12.SD_DIN, U$12.T_DIN
- net TXD: now also U$1.DIO_18, U$12.TXD; no longer IC1.TXD, U$1.DIO_30
- net VUSB_IN: now also C30.1, C31.1, U$12.VCC
- net V_DISP: now also U$14.VCC0, U$14.VCC1; no longer U$12.RD, U$12.VCC
- net V_USB: no longer C31.1, C32.1, IC1.VCC
Other:
- moved on the sheet: C30, C31, C32
