File: eagle/badge2016.sch (EAGLE design)
At the start: 121 parts, among them IC1 25AA080SN, IC2 FT231XQ, J1 USB-MICRO, Q2 BC857ALT1SMD, Q2_24MHZ NX5032G, X1 PASSER-07, X10 PAD-1.27X1.27, X11 PAD-1.27X1.27, X12 PAD-1.27X1.27, X13 PAD-1.27X1.27, X14 PAD-1.27X1.27, X15 PAD-1.27X1.27, X16 PAD-1.27X1.27, X17 PAD-1.27X1.27, X18 PAD-1.27X1.27, X19 PAD-1.27X1.27, X2 PASSER-07, X20 PAD-1.27X1.27, X21 PAD-0.5, X3 PASSER-07, X4 PAD-0.5, X5 PAD-0.5, X6 PAD-0.5, X7 PAD-0.5, X8 PAD-1.27X1.27, X9 PAD-1.27X1.27

Commit message: fixed serial lines optimized ground layer below cc1310 changed ltc footprint, less cream fixed missing v_usb line below usb socket
Parts:
- renumbered R15 to NC_R18, R16 to NC_R19
Connections:
- removed net RXD: IC2.RXD, NC-UART.5, NC_R19.2
- removed net TXD: IC2.TXD, NC-UART.4, NC_R18.2
- removed net UART_RXD: NC_R18.1, U$1.DIO_2
- removed net UART_TXD: NC_R19.1, U$1.DIO_3
- new net FTDI_RXD: IC2.RXD, NC-UART.5, NC_R19.1, NC_R19.2, U$1.DIO_3
- new net FTDI_TXD: IC2.TXD, NC-UART.4, NC_R18.1, NC_R18.2, U$1.DIO_2
Changed lines of the file:
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@@
 <?xml version="1.0" encoding="utf-8"?>
 <!DOCTYPE eagle SYSTEM "eagle.dtd">
-<eagle version="7.3.0">
+<eagle version="7.5.0">
 <drawing>
 <settings>
@@
 <part name="GND28" library="supply1" deviceset="GND" device=""/>
 <part name="X21" library="we-rcl" deviceset="PAD" device="-0.5"/>
-<part name="R15" library="we-rcl" deviceset="RESISTOR" device="-0402" value="0"/>
-<part name="R16" library="we-rcl" deviceset="RESISTOR" device="-0402" value="0"/>
+<part name="NC_R18" library="we-rcl" deviceset="RESISTOR" device="-0402" value="0"/>
+<part name="NC_R19" library="we-rcl" deviceset="RESISTOR" device="-0402" value="0"/>
 </parts>
 <sheets>
@@
 <instance part="GND28" gate="1" x="-7.62" y="-386.08" rot="R270"/>
 <instance part="X21" gate="X" x="45.72" y="-10.16" rot="R90"/>
-<instance part="R15" gate="R" x="-185.42" y="-436.88" rot="R180"/>
-<instance part="R16" gate="R" x="-177.8" y="-439.42" rot="R180"/>
+<instance part="NC_R18" gate="R" x="-185.42" y="-436.88" rot="R180"/>
+<instance part="NC_R19" gate="R" x="-177.8" y="-439.42" rot="R180"/>
 </instances>
 <busses>
@@
 </segment>
 </net>
-<net name="TXD" class="0">
-<segment>
-<pinref part="IC2" gate="IC" pin="TXD"/>
-<wire x1="-205.74" y1="-436.88" x2="-190.5" y2="-436.88" width="0.1524" layer="91"/>
-<label x="-200.66" y="-436.88" size="1.778" layer="95"/>
-<pinref part="R15" gate="R" pin="2"/>
-</segment>
-<segment>
-<pinref part="NC-UART" gate="A" pin="4"/>
-<wire x1="187.96" y1="251.46" x2="223.52" y2="251.46" width="0.1524" layer="91"/>
-<label x="193.04" y="251.46" size="1.778" layer="95"/>
-</segment>
-</net>
 <net name="I2C_SDA" class="0">
 <segment>
@@
 <pinref part="X5" gate="X" pin="P"/>
 <wire x1="91.44" y1="45.72" x2="111.76" y2="45.72" width="0.1524" layer="91"/>
-<wire x1="114.3" y1="45.72" x2="111.76" y2="45.72" width="0.1524" layer="91"/>
 </segment>
 </net>
@@
 </segment>
 </net>
-<net name="RXD" class="0">
+<net name="FTDI_RXD" class="0">
 <segment>
 <pinref part="IC2" gate="IC" pin="RXD"/>
 <wire x1="-205.74" y1="-439.42" x2="-182.88" y2="-439.42" width="0.1524" layer="91"/>
 <label x="-200.66" y="-439.42" size="1.778" layer="95"/>
-<pinref part="R16" gate="R" pin="2"/>
+<pinref part="NC_R19" gate="R" pin="2"/>
+<pinref part="NC_R19" gate="R" pin="1"/>
+<wire x1="-172.72" y1="-439.42" x2="-165.1" y2="-439.42" width="0.1524" layer="91"/>
+<wire x1="-182.88" y1="-439.42" x2="-172.72" y2="-439.42" width="0.1524" layer="91"/>
+<junction x="-182.88" y="-439.42"/>
+<junction x="-172.72" y="-439.42"/>
 </segment>
 <segment>
@@
 <label x="193.04" y="248.92" size="1.778" layer="95"/>
 </segment>
-</net>
-<net name="UART_RXD" class="0">
+<segment>
+<pinref part="U$1" gate="G$1" pin="DIO_3"/>
+<wire x1="22.86" y1="38.1" x2="0" y2="38.1" width="0.1524" layer="91"/>
+<label x="2.54" y="38.1" size="1.778" layer="95"/>
+</segment>
+</net>
+<net name="FTDI_TXD" class="0">
 <segment>
 <pinref part="U$1" gate="G$1" pin="DIO_2"/>
@@
 </segment>
 <segment>
-<pinref part="R15" gate="R" pin="1"/>
+<pinref part="IC2" gate="IC" pin="TXD"/>
+<wire x1="-205.74" y1="-436.88" x2="-190.5" y2="-436.88" width="0.1524" layer="91"/>
+<label x="-200.66" y="-436.88" size="1.778" layer="95"/>
+<pinref part="NC_R18" gate="R" pin="2"/>
+<pinref part="NC_R18" gate="R" pin="1"/>
 <wire x1="-180.34" y1="-436.88" x2="-165.1" y2="-436.88" width="0.1524" layer="91"/>
-</segment>
-</net>
-<net name="UART_TXD" class="0">
-<segment>
-<pinref part="U$1" gate="G$1" pin="DIO_3"/>
-<wire x1="22.86" y1="38.1" x2="0" y2="38.1" width="0.1524" layer="91"/>
-<label x="2.54" y="38.1" size="1.778" layer="95"/>
-</segment>
-<segment>
-<pinref part="R16" gate="R" pin="1"/>
-<wire x1="-172.72" y1="-439.42" x2="-165.1" y2="-439.42" width="0.1524" layer="91"/>
-</segment>
-</net>
+<wire x1="-190.5" y1="-436.88" x2="-180.34" y2="-436.88" width="0.1524" layer="91"/>
+<junction x="-190.5" y="-436.88"/>
+<junction x="-180.34" y="-436.88"/>
+</segment>
+<segment>
+<pinref part="NC-UART" gate="A" pin="4"/>
+<wire x1="187.96" y1="251.46" x2="223.52" y2="251.46" width="0.1524" layer="91"/>
+<label x="193.04" y="251.46" size="1.778" layer="95"/>
+</segment>
+</net>

Commit message: fixes ski
Parts:
- added C36: 100µF, we-rcl:CAPACITOR-1206
- added R15: 0R3, we-rcl:RESISTOR-0402
Connections:
- new net N$54: C36.2, R15.1
- net GND: now also R15.2
- net N$20: now also C36.1
Changed lines of the file:
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@@
 <part name="NC_R18" library="we-rcl" deviceset="RESISTOR" device="-0402" value="0"/>
 <part name="NC_R19" library="we-rcl" deviceset="RESISTOR" device="-0402" value="0"/>
+<part name="C36" library="we-rcl" deviceset="CAPACITOR" device="-1206" value="100µF"/>
+<part name="R15" library="we-rcl" deviceset="RESISTOR" device="-0402" value="0R3"/>
+<part name="GND53" library="supply1" deviceset="GND" device=""/>
 </parts>
 <sheets>
@@
 <instance part="NC_R18" gate="R" x="-185.42" y="-436.88" rot="R180"/>
 <instance part="NC_R19" gate="R" x="-177.8" y="-439.42" rot="R180"/>
+<instance part="C36" gate="C" x="35.56" y="-264.16"/>
+<instance part="R15" gate="R" x="45.72" y="-264.16"/>
+<instance part="GND53" gate="1" x="55.88" y="-264.16" rot="R90"/>
 </instances>
 <busses>
@@
 <wire x1="10.16" y1="-386.08" x2="-5.08" y2="-386.08" width="0.1524" layer="91"/>
 </segment>
+<segment>
+<pinref part="GND53" gate="1" pin="GND"/>
+<pinref part="R15" gate="R" pin="2"/>
+<wire x1="53.34" y1="-264.16" x2="50.8" y2="-264.16" width="0.1524" layer="91"/>
+</segment>
 </net>
 <net name="3V3" class="0">
@@
 <segment>
 <pinref part="U$11" gate="G$1" pin="BAT"/>
-<wire x1="25.4" y1="-307.34" x2="25.4" y2="-256.54" width="0.1524" layer="91"/>
+<wire x1="25.4" y1="-307.34" x2="25.4" y2="-264.16" width="0.1524" layer="91"/>
 <pinref part="NC-JP2" gate="G$1" pin="1"/>
+<wire x1="25.4" y1="-264.16" x2="25.4" y2="-256.54" width="0.1524" layer="91"/>
 <wire x1="25.4" y1="-256.54" x2="45.72" y2="-256.54" width="0.1524" layer="91"/>
 <wire x1="45.72" y1="-256.54" x2="45.72" y2="-246.38" width="0.1524" layer="91"/>
@@
 <wire x1="17.78" y1="-256.54" x2="17.78" y2="-248.92" width="0.1524" layer="91"/>
 <junction x="25.4" y="-256.54"/>
+<pinref part="C36" gate="C" pin="1"/>
+<wire x1="33.02" y1="-264.16" x2="25.4" y2="-264.16" width="0.1524" layer="91"/>
+<junction x="25.4" y="-264.16"/>
 </segment>
 </net>
@@
 </segment>
 </net>
+<net name="N$54" class="0">
+<segment>
+<pinref part="R15" gate="R" pin="1"/>
+<pinref part="C36" gate="C" pin="2"/>
+<wire x1="40.64" y1="-264.16" x2="38.1" y2="-264.16" width="0.1524" layer="91"/>
+</segment>
+</net>

Commit message: newest pcb state
Parts:
- added NC_BLBD_3V3, NC_BLBD_GND, NC_BLBD_PD, NC_BLBD_PU: (no value), we-rcl:RESISTOR-0402
- added NC_BOOTLOADER_BTN: KSEM31G, ERNW_parts:KSEM31G
Connections:
- removed net N$38: U$1.DIO_20, X7.P
- new net BOOTLOADER_BACKDOOR: NC_BLBD_PD.2, NC_BLBD_PU.2, NC_BOOTLOADER_BTN.B1, NC_BOOTLOADER_BTN.B2, U$1.DIO_20, X7.P
- new net N$55: NC_BLBD_3V3.2, NC_BLBD_GND.2, NC_BOOTLOADER_BTN.A1, NC_BOOTLOADER_BTN.A2
- net 3V3: now also NC_BLBD_3V3.1, NC_BLBD_PU.1
- net GND: now also NC_BLBD_GND.1, NC_BLBD_PD.1
Other:
- moved on the sheet: X7
Changed lines of the file:
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@@
 <part name="R15" library="we-rcl" deviceset="RESISTOR" device="-0402" value="0R3"/>
 <part name="GND53" library="supply1" deviceset="GND" device=""/>
+<part name="NC_BOOTLOADER_BTN" library="ERNW_parts" deviceset="KSEM31G" device=""/>
+<part name="NC_BLBD_PD" library="we-rcl" deviceset="RESISTOR" device="-0402"/>
+<part name="NC_BLBD_PU" library="we-rcl" deviceset="RESISTOR" device="-0402"/>
+<part name="NC_BLBD_GND" library="we-rcl" deviceset="RESISTOR" device="-0402"/>
+<part name="NC_BLBD_3V3" library="we-rcl" deviceset="RESISTOR" device="-0402"/>
+<part name="GND59" library="supply1" deviceset="GND" device=""/>
+<part name="GND60" library="supply1" deviceset="GND" device=""/>
 </parts>
 <sheets>
@@
 <instance part="X5" gate="X" x="114.3" y="45.72" rot="R180"/>
 <instance part="X6" gate="X" x="114.3" y="43.18" rot="R180"/>
-<instance part="X7" gate="X" x="114.3" y="40.64" rot="R180"/>
+<instance part="X7" gate="X" x="129.54" y="43.18" rot="R270"/>
 <instance part="X8" gate="X" x="-142.24" y="-269.24" rot="R90"/>
 <instance part="X9" gate="X" x="-142.24" y="-261.62" rot="R270"/>
@@
 <instance part="R15" gate="R" x="45.72" y="-264.16"/>
 <instance part="GND53" gate="1" x="55.88" y="-264.16" rot="R90"/>
+<instance part="NC_BOOTLOADER_BTN" gate="G$1" x="170.18" y="12.7" rot="R180"/>
+<instance part="NC_BLBD_PD" gate="R" x="137.16" y="2.54" rot="R90"/>
+<instance part="NC_BLBD_PU" gate="R" x="144.78" y="2.54" rot="R90"/>
+<instance part="NC_BLBD_GND" gate="R" x="190.5" y="2.54" rot="R90"/>
+<instance part="NC_BLBD_3V3" gate="R" x="198.12" y="2.54" rot="R90"/>
+<instance part="GND59" gate="1" x="137.16" y="-10.16"/>
+<instance part="GND60" gate="1" x="190.5" y="-10.16"/>
 </instances>
 <busses>
@@
 <wire x1="53.34" y1="-264.16" x2="50.8" y2="-264.16" width="0.1524" layer="91"/>
 </segment>
+<segment>
+<pinref part="NC_BLBD_PD" gate="R" pin="1"/>
+<pinref part="GND59" gate="1" pin="GND"/>
+<wire x1="137.16" y1="-2.54" x2="137.16" y2="-7.62" width="0.1524" layer="91"/>
+</segment>
+<segment>
+<pinref part="NC_BLBD_GND" gate="R" pin="1"/>
+<pinref part="GND60" gate="1" pin="GND"/>
+<wire x1="190.5" y1="-2.54" x2="190.5" y2="-7.62" width="0.1524" layer="91"/>
+</segment>
 </net>
 <net name="3V3" class="0">
@@
 <wire x1="218.44" y1="-187.96" x2="218.44" y2="-185.42" width="0.1524" layer="91"/>
 <junction x="218.44" y="-185.42"/>
+</segment>
+<segment>
+<pinref part="NC_BLBD_PU" gate="R" pin="1"/>
+<wire x1="144.78" y1="-2.54" x2="144.78" y2="-10.16" width="0.1524" layer="91"/>
+<label x="144.78" y="-7.62" size="1.778" layer="95" rot="R90"/>
+</segment>
+<segment>
+<pinref part="NC_BLBD_3V3" gate="R" pin="1"/>
+<wire x1="198.12" y1="-2.54" x2="198.12" y2="-10.16" width="0.1524" layer="91"/>
+<label x="198.12" y="-7.62" size="1.778" layer="95" rot="R90"/>
 </segment>
 </net>
@@
 </segment>
 </net>
-<net name="N$38" class="0">
+<net name="BOOTLOADER_BACKDOOR" class="0">
 <segment>
 <pinref part="U$1" gate="G$1" pin="DIO_20"/>
 <pinref part="X7" gate="X" pin="P"/>
-<wire x1="91.44" y1="40.64" x2="111.76" y2="40.64" width="0.1524" layer="91"/>
+<wire x1="91.44" y1="40.64" x2="129.54" y2="40.64" width="0.1524" layer="91"/>
+<wire x1="129.54" y1="40.64" x2="137.16" y2="40.64" width="0.1524" layer="91"/>
+<wire x1="137.16" y1="40.64" x2="137.16" y2="15.24" width="0.1524" layer="91"/>
+<junction x="129.54" y="40.64"/>
+<pinref part="NC_BOOTLOADER_BTN" gate="G$1" pin="B2"/>
+<wire x1="137.16" y1="15.24" x2="144.78" y2="15.24" width="0.1524" layer="91"/>
+<pinref part="NC_BLBD_PD" gate="R" pin="2"/>
+<wire x1="144.78" y1="15.24" x2="157.48" y2="15.24" width="0.1524" layer="91"/>
+<wire x1="137.16" y1="15.24" x2="137.16" y2="7.62" width="0.1524" layer="91"/>
+<junction x="137.16" y="15.24"/>
+<pinref part="NC_BLBD_PU" gate="R" pin="2"/>
+<wire x1="144.78" y1="15.24" x2="144.78" y2="7.62" width="0.1524" layer="91"/>
+<junction x="144.78" y="15.24"/>
+<pinref part="NC_BOOTLOADER_BTN" gate="G$1" pin="B1"/>
+<wire x1="157.48" y1="15.24" x2="157.48" y2="10.16" width="0.1524" layer="91"/>
+<junction x="157.48" y="15.24"/>
+<label x="96.52" y="40.64" size="1.778" layer="95"/>
 </segment>
 </net>
@@
 </segment>
 </net>
+<net name="N$55" class="0">
+<segment>
+<pinref part="NC_BOOTLOADER_BTN" gate="G$1" pin="A1"/>
+<pinref part="NC_BLBD_GND" gate="R" pin="2"/>
+<wire x1="182.88" y1="10.16" x2="190.5" y2="10.16" width="0.1524" layer="91"/>
+<wire x1="190.5" y1="10.16" x2="190.5" y2="7.62" width="0.1524" layer="91"/>
+<pinref part="NC_BLBD_3V3" gate="R" pin="2"/>
+<wire x1="190.5" y1="10.16" x2="198.12" y2="10.16" width="0.1524" layer="91"/>
+<wire x1="198.12" y1="10.16" x2="198.12" y2="7.62" width="0.1524" layer="91"/>
+<junction x="190.5" y="10.16"/>
+<pinref part="NC_BOOTLOADER_BTN" gate="G$1" pin="A2"/>
+<wire x1="182.88" y1="15.24" x2="182.88" y2="10.16" width="0.1524" layer="91"/>
+<junction x="182.88" y="10.16"/>
+</segment>
+</net>

Commit message: final pcb layout + schematic
Parts:
- removed NC_BLBD_3V3, NC_BLBD_GND, NC_BLBD_PU: (no value), we-rcl:RESISTOR-0402
- removed X11, X8, X9: PAD-1.27X1.27, we-rcl:PAD-1.27X1.27
- added U$7: YELLOW_BUSH, ERNW_parts:YELLOW_BUSH
- B_LOADER_PDWN: value (none) -> 10k
- L1: device we-rcl:INDUCTOR-0402 -> we-rcl:INDUCTOR-0603
- renumbered NC-U$13 to BTN_RESET, NC_BLBD_PD to B_LOADER_PDWN, NC_BOOTLOADER_BTN to BOOTLOADER_BTN, R13 to NC_R13, R14 to NC_R14
Connections:
- removed net N$33: NC_R14.1, U$11.PGOOD
- removed net N$55: BOOTLOADER_BTN.A1, BOOTLOADER_BTN.A2, NC_BLBD_3V3.2, NC_BLBD_GND.2
- net 3V3: now also BOOTLOADER_BTN.A1, BOOTLOADER_BTN.A2; no longer NC_BLBD_3V3.1, NC_BLBD_PU.1
- net BOOTLOADER_BACKDOOR: no longer NC_BLBD_PU.2
- net GND: no longer NC_BLBD_GND.1, X11.P
- net N$25: no longer X8.P
- net N$30: now also NC_R14.1, U$11.PGOOD
- net N$32: no longer X9.P

Commit message: Final Badge!
Parts:
- added R13, R14: 100k, we-rcl:RESISTOR-0402
Connections:
- new net N$33: IC1.!HOLD, R14.2
- new net N$38: IC1.!WP, R13.2
- net 3V3: now also R13.1, R14.1
Changed lines of the file:
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@@
 <part name="GND59" library="supply1" deviceset="GND" device=""/>
 <part name="U$7" library="ERNW_parts" deviceset="YELLOW_BUSH" device=""/>
+<part name="R13" library="we-rcl" deviceset="RESISTOR" device="-0402" value="100k"/>
+<part name="R14" library="we-rcl" deviceset="RESISTOR" device="-0402" value="100k"/>
 </parts>
 <sheets>
@@
 <instance part="GND59" gate="1" x="137.16" y="-10.16"/>
 <instance part="U$7" gate="G$1" x="-50.8" y="-149.86"/>
+<instance part="R13" gate="R" x="264.16" y="-66.04" rot="R270"/>
+<instance part="R14" gate="R" x="256.54" y="-66.04" rot="R270"/>
 </instances>
 <busses>
@@
 <segment>
 <pinref part="IC1" gate="G$1" pin="VCC"/>
-<wire x1="287.02" y1="-68.58" x2="287.02" y2="-58.42" width="0.1524" layer="91"/>
+<wire x1="287.02" y1="-68.58" x2="287.02" y2="-60.96" width="0.1524" layer="91"/>
 <label x="287.02" y="-66.04" size="1.778" layer="95" rot="R90"/>
+<wire x1="287.02" y1="-60.96" x2="287.02" y2="-58.42" width="0.1524" layer="91"/>
+<wire x1="256.54" y1="-60.96" x2="264.16" y2="-60.96" width="0.1524" layer="91"/>
+<junction x="287.02" y="-60.96"/>
+<pinref part="R13" gate="R" pin="1"/>
+<wire x1="264.16" y1="-60.96" x2="287.02" y2="-60.96" width="0.1524" layer="91"/>
+<junction x="264.16" y="-60.96"/>
+<pinref part="R14" gate="R" pin="1"/>
 </segment>
 <segment>
@@
 </segment>
 </net>
+<net name="N$33" class="0">
+<segment>
+<pinref part="IC1" gate="G$1" pin="!HOLD"/>
+<wire x1="266.7" y1="-86.36" x2="256.54" y2="-86.36" width="0.1524" layer="91"/>
+<wire x1="256.54" y1="-86.36" x2="256.54" y2="-71.12" width="0.1524" layer="91"/>
+<pinref part="R14" gate="R" pin="2"/>
+</segment>
+</net>
+<net name="N$38" class="0">
+<segment>
+<pinref part="IC1" gate="G$1" pin="!WP"/>
+<wire x1="266.7" y1="-73.66" x2="264.16" y2="-73.66" width="0.1524" layer="91"/>
+<wire x1="264.16" y1="-73.66" x2="264.16" y2="-71.12" width="0.1524" layer="91"/>
+<pinref part="R13" gate="R" pin="2"/>
+</segment>
+</net>
