File: eagle/badge2016.sch (EAGLE design)
At the start: 125 parts, among them IC1 25AA080SN, IC2 FT231XQ, J1 USB-MICRO, Q2 BC857ALT1SMD, Q2_24MHZ NX5032G, X1 PASSER-07, X10 PAD-1.27X1.27, X12 PAD-1.27X1.27, X13 PAD-1.27X1.27, X14 PAD-1.27X1.27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

Commit message: fixed final values in schematics: changed spi memory to 1M change loads of caps
Parts:
- 25AA1024T: value 25AA080SN -> 25AA1024T
- renumbered IC1 to 25AA1024T
Changed lines of the file:
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@@
 <part name="R20" library="we-rcl" deviceset="RESISTOR" device="-0402" value="1k5"/>
 <part name="U$15" library="ERNW_parts" deviceset="JST-2" device=""/>
-<part name="IC1" library="microchip" deviceset="25*" device="SN" technology="AA080"/>
+<part name="25AA1024T" library="microchip" deviceset="25*" device="SN" technology="AA080" value="25AA1024T"/>
 <part name="GND56" library="supply1" deviceset="GND" device=""/>
 <part name="NC-R15" library="we-rcl" deviceset="RESISTOR" device="-0402" value="NC"/>
@@
 <instance part="R20" gate="R" x="-167.64" y="-459.74" rot="R180"/>
 <instance part="U$15" gate="G$1" x="22.86" y="-238.76"/>
-<instance part="IC1" gate="G$1" x="279.4" y="-81.28"/>
+<instance part="25AA1024T" gate="G$1" x="279.4" y="-81.28"/>
 <instance part="GND56" gate="1" x="287.02" y="-99.06"/>
 <instance part="NC-R15" gate="R" x="218.44" y="-193.04" rot="R270"/>
@@
 </segment>
 <segment>
-<pinref part="IC1" gate="G$1" pin="GND"/>
+<pinref part="25AA1024T" gate="G$1" pin="GND"/>
 <pinref part="GND56" gate="1" pin="GND"/>
 <wire x1="287.02" y1="-91.44" x2="287.02" y2="-96.52" width="0.1524" layer="91"/>
@@
 </segment>
 <segment>
-<pinref part="IC1" gate="G$1" pin="VCC"/>
+<pinref part="25AA1024T" gate="G$1" pin="VCC"/>
 <wire x1="287.02" y1="-68.58" x2="287.02" y2="-60.96" width="0.1524" layer="91"/>
 <label x="287.02" y="-66.04" size="1.778" layer="95" rot="R90"/>
@@
 </segment>
 <segment>
-<pinref part="IC1" gate="G$1" pin="SI"/>
+<pinref part="25AA1024T" gate="G$1" pin="SI"/>
 <wire x1="266.7" y1="-81.28" x2="248.92" y2="-81.28" width="0.1524" layer="91"/>
 <label x="251.46" y="-81.28" size="1.778" layer="95"/>
 </segment>
 <segment>
-<pinref part="IC1" gate="G$1" pin="SO"/>
+<pinref part="25AA1024T" gate="G$1" pin="SO"/>
 <wire x1="294.64" y1="-81.28" x2="309.88" y2="-81.28" width="0.1524" layer="91"/>
 <label x="297.18" y="-81.28" size="1.778" layer="95"/>
@@
 </segment>
 <segment>
-<pinref part="IC1" gate="G$1" pin="SCK"/>
+<pinref part="25AA1024T" gate="G$1" pin="SCK"/>
 <wire x1="266.7" y1="-83.82" x2="248.92" y2="-83.82" width="0.1524" layer="91"/>
 <label x="251.46" y="-83.82" size="1.778" layer="95"/>
@@
 <net name="EEPROM_!CS" class="0">
 <segment>
-<pinref part="IC1" gate="G$1" pin="!CS"/>
+<pinref part="25AA1024T" gate="G$1" pin="!CS"/>
 <wire x1="266.7" y1="-78.74" x2="248.92" y2="-78.74" width="0.1524" layer="91"/>
 <label x="251.46" y="-78.74" size="1.778" layer="95"/>
@@
 <net name="N$33" class="0">
 <segment>
-<pinref part="IC1" gate="G$1" pin="!HOLD"/>
+<pinref part="25AA1024T" gate="G$1" pin="!HOLD"/>
 <wire x1="266.7" y1="-86.36" x2="256.54" y2="-86.36" width="0.1524" layer="91"/>
 <wire x1="256.54" y1="-86.36" x2="256.54" y2="-71.12" width="0.1524" layer="91"/>
@@
 <net name="N$38" class="0">
 <segment>
-<pinref part="IC1" gate="G$1" pin="!WP"/>
+<pinref part="25AA1024T" gate="G$1" pin="!WP"/>
 <wire x1="266.7" y1="-73.66" x2="264.16" y2="-73.66" width="0.1524" layer="91"/>
 <wire x1="264.16" y1="-73.66" x2="264.16" y2="-71.12" width="0.1524" layer="91"/>

Commit message: changed values of NC parts so that they'd appear in BOM added final BOM as sent to watterott
Parts:
- NC-R16, NC-R17, NC_R13: value 10k -> NC_10k
- NC_C35: value 100nF -> NC_100nF
- NC_C36: value 4.7µF -> NC_4.7µF
- NC_R14: value 0R -> NC_0R
- NC_R15, NC_R16, NC_R2, NC_R3: value 0 -> NC_0R
- NC_R18, NC_R19: value 0 -> NC_0
- NC_R5: value 1k5 -> NC_1k5
Changed lines of the file:
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@@
 <part name="GND18" library="supply1" deviceset="GND" device=""/>
 <part name="GND19" library="supply1" deviceset="GND" device=""/>
-<part name="NC_R2" library="we-rcl" deviceset="RESISTOR" device="-0603" value="0"/>
-<part name="NC_R3" library="we-rcl" deviceset="RESISTOR" device="-0603" value="0"/>
+<part name="NC_R2" library="we-rcl" deviceset="RESISTOR" device="-0603" value="NC_0R"/>
+<part name="NC_R3" library="we-rcl" deviceset="RESISTOR" device="-0603" value="NC_0R"/>
 <part name="L9" library="we-rcl" deviceset="INDUCTOR" device="-0402" value="12nH"/>
 <part name="C22" library="we-rcl" deviceset="CAPACITOR" device="-0402" value="1pF"/>
@@
 <part name="GND45" library="supply1" deviceset="GND" device=""/>
 <part name="R12" library="we-rcl" deviceset="RESISTOR" device="-0402" value="0R"/>
-<part name="NC_R13" library="we-rcl" deviceset="RESISTOR" device="-0402" value="10k"/>
+<part name="NC_R13" library="we-rcl" deviceset="RESISTOR" device="-0402" value="NC_10k"/>
 <part name="GND46" library="supply1" deviceset="GND" device=""/>
-<part name="NC_R14" library="we-rcl" deviceset="RESISTOR" device="-0402" value="0R"/>
+<part name="NC_R14" library="we-rcl" deviceset="RESISTOR" device="-0402" value="NC_0R"/>
 <part name="NC-IC3" library="microchip" deviceset="24*" device="SN" technology="AA01"/>
 <part name="GND47" library="supply1" deviceset="GND" device=""/>
@@
 <part name="GND49" library="supply1" deviceset="GND" device=""/>
 <part name="GND50" library="supply1" deviceset="GND" device=""/>
-<part name="NC-R16" library="we-rcl" deviceset="RESISTOR" device="-0402" value="10k"/>
-<part name="NC-R17" library="we-rcl" deviceset="RESISTOR" device="-0402" value="10k"/>
+<part name="NC-R16" library="we-rcl" deviceset="RESISTOR" device="-0402" value="NC_10k"/>
+<part name="NC-R17" library="we-rcl" deviceset="RESISTOR" device="-0402" value="NC_10k"/>
 <part name="NC-JP4" library="pinhead" deviceset="PINHD-2X8" device=""/>
 <part name="GND51" library="supply1" deviceset="GND" device=""/>
@@
 <part name="NC-SD1" library="we-con" deviceset="SD-CARD" device="-MSD50"/>
 <part name="GND40" library="supply1" deviceset="GND" device=""/>
-<part name="NC_C35" library="we-rcl" deviceset="CAPACITOR" device="-0402" value="100nF"/>
-<part name="NC_C36" library="we-rcl" deviceset="CAPACITOR" device="-0402" value="4.7µF"/>
+<part name="NC_C35" library="we-rcl" deviceset="CAPACITOR" device="-0402" value="NC_100nF"/>
+<part name="NC_C36" library="we-rcl" deviceset="CAPACITOR" device="-0402" value="NC_4.7µF"/>
 <part name="GND41" library="supply1" deviceset="GND" device=""/>
 <part name="GND54" library="supply1" deviceset="GND" device=""/>
@@
 <part name="U$6" library="ERNW_parts" deviceset="TR_PIGPEN" device=""/>
 <part name="LOGO1" library="we-symbol" deviceset="LOGO" device="-S_LAYER"/>
-<part name="NC_R15" library="we-rcl" deviceset="RESISTOR" device="-0603" value="0"/>
-<part name="NC_R16" library="we-rcl" deviceset="RESISTOR" device="-0603" value="0"/>
+<part name="NC_R15" library="we-rcl" deviceset="RESISTOR" device="-0603" value="NC_0R"/>
+<part name="NC_R16" library="we-rcl" deviceset="RESISTOR" device="-0603" value="NC_0R"/>
 <part name="X4" library="we-rcl" deviceset="PAD" device="-0.5"/>
 <part name="X5" library="we-rcl" deviceset="PAD" device="-0.5"/>
@@
 <part name="X17" library="we-rcl" deviceset="PAD" device="-1.27X1.27"/>
 <part name="NC_LED2" library="we-opto" deviceset="LED" device="-0603"/>
-<part name="NC_R5" library="we-rcl" deviceset="RESISTOR" device="-0402" value="1k5"/>
+<part name="NC_R5" library="we-rcl" deviceset="RESISTOR" device="-0402" value="NC_1k5"/>
 <part name="GND52" library="supply1" deviceset="GND" device=""/>
 <part name="X18" library="we-rcl" deviceset="PAD" device="-1.27X1.27"/>
@@
 <part name="GND28" library="supply1" deviceset="GND" device=""/>
 <part name="X21" library="we-rcl" deviceset="PAD" device="-0.5"/>
-<part name="NC_R18" library="we-rcl" deviceset="RESISTOR" device="-0402" value="0"/>
-<part name="NC_R19" library="we-rcl" deviceset="RESISTOR" device="-0402" value="0"/>
+<part name="NC_R18" library="we-rcl" deviceset="RESISTOR" device="-0402" value="NC_0"/>
+<part name="NC_R19" library="we-rcl" deviceset="RESISTOR" device="-0402" value="NC_0"/>
 <part name="C36" library="we-rcl" deviceset="CAPACITOR" device="-1206" value="100µF"/>
 <part name="R15" library="we-rcl" deviceset="RESISTOR" device="-0402" value="0R3"/>
